File: miditerm/miditerm.kicad_pcb (KiCad board)
At the start: 2 copper layers, 60 x 30 mm, 51 parts, among them J1 USB, J2 MIDI IN, J3 MIDI OUT, J4 GND, U1 USBLC6-2SC6, U2 FT231XS, U3 H11L1

Commit message: Cleanup
Routing:
- net GND: track 23.3 -> 23.1 mm, vias 104 -> 103
